File: dsn-vc288-v2/dsn-vc288-v2.sch (KiCad schematic (older format))
At the start: 25 parts, among them IC1 ME6203, IC2 STM8S103F3, IC3 LM358, J1 Programming Port 1, J2 Programming Port 2, J3 Conn_01x03, J4 Conn_01x02

Commit message: Updated directory sturcture and changed V2 schematics to KiCAD 5.
Parts:
- C1, C2, C3, C4: symbol C -> V2-DSN-VC288-rescue:C
- D1: symbol D_ALT -> V2-DSN-VC288-rescue:D_ALT
- DS1, DS2: symbol MCD-2831A -> mcd-2831a:MCD-2831A
- IC1: symbol ME6203 -> me6203:ME6203
- IC2: symbol STM8S103F3 -> stm8s103f3:STM8S103F3
- IC3: symbol LM358 -> V2-DSN-VC288-rescue:LM358
- J1: symbol Conn_01x08 -> V2-DSN-VC288-rescue:CONN_01X08
- J2, J4: symbol Conn_01x02 -> V2-DSN-VC288-rescue:CONN_01X02
- J3: symbol Conn_01x03 -> V2-DSN-VC288-rescue:CONN_01X03
- R1, R2, R3, R4, R5, R6: symbol R -> V2-DSN-VC288-rescue:R
- RN1, RN2: symbol R_Pack04 -> V2-DSN-VC288-rescue:R_Pack04
- RV1, RV2: symbol POT_TRIM -> V2-DSN-VC288-rescue:POT_TRIM
- SH-R1: symbol ShuntResistor -> ShuntResistor:ShuntResistor
Connections:
- wire segments 185 -> 209
